Commit message: testing own robot

File: urdf/test.xacro (robot description, xacro)
@@ -5,98 +5,5 @@
 <!-- =================================================================================== -->
 <robot name="udacity_bot" xmlns:xacro="http://www.ros.org/wiki/xacro">
-  <gazebo>
-    <plugin filename="libgazebo_ros_diff_drive.so" name="differential_drive_controller">
-      <legacyMode>false</legacyMode>
-      <alwaysOn>true</alwaysOn>
-      <updateRate>10</updateRate>
-      <leftJoint>left_wheel_hinge</leftJoint>
-      <rightJoint>right_wheel_hinge</rightJoint>
-      <wheelSeparation>0.4</wheelSeparation>
-      <wheelDiameter>0.2</wheelDiameter>
-      <torque>10</torque>
-      <commandTopic>cmd_vel</commandTopic>
-      <odometryTopic>odom</odometryTopic>
-      <odometryFrame>odom</odometryFrame>
-      <robotBaseFrame>robot_footprint</robotBaseFrame>
-    </plugin>
-  </gazebo>
-  <gazebo reference="camera">
-    <material name="gold">
-      <color rgba="1 0.549 0 1"/>
-    </material>
-    <sensor name="camera1" type="camera">
-      <update_rate>30.0</update_rate>
-      <camera name="head">
-        <horizontal_fov>1.3962634</horizontal_fov>
-        <image>
-          <width>800</width>
-          <height>800</height>
-          <format>R8G8B8</format>
-        </image>
-        <clip>
-          <near>0.02</near>
-          <far>300</far>
-        </clip>
-      </camera>
-      <plugin filename="libgazebo_ros_camera.so" name="camera_controller">
-        <alwaysOn>true</alwaysOn>
-        <updateRate>0.0</updateRate>
-        <cameraName>udacity_bot/camera1</cameraName>
-        <imageTopicName>image_raw</imageTopicName>
-        <cameraInfoTopicName>camera_info</cameraInfoTopicName>
-        <frameName>camera</frameName>
-        <hackBaseline>0.07</hackBaseline>
-        <distortionK1>0.0</distortionK1>
-        <distortionK2>0.0</distortionK2>
-        <distortionK3>0.0</distortionK3>
-        <distortionT1>0.0</distortionT1>
-        <distortionT2>0.0</distortionT2>
-      </plugin>
-    </sensor>
-  </gazebo>
-  <!-- hokuyo -->
-  <gazebo reference="hokuyo">
-    <sensor name="head_hokuyo_sensor" type="ray">
-      <pose>0 0 0 0 0 0</pose>
-      <visualize>false</visualize>
-      <update_rate>40</update_rate>
-      <ray>
-        <scan>
-          <horizontal>
-            <samples>720</samples>
-            <resolution>1</resolution>
-            <min_angle>-1.570796</min_angle>
-            <max_angle>1.570796</max_angle>
-          </horizontal>
-        </scan>
-        <range>
-          <min>0.10</min>
-          <max>30.0</max>
-          <resolution>0.01</resolution>
-        </range>
-        <noise>
-          <type>gaussian</type>
-          <!-- Noise parameters based on published spec for Hokuyo laser
-               achieving "+-30mm" accuracy at range < 10m.  A mean of 0.0m and
-               stddev of 0.01m will put 99.7% of samples within 0.03m of the true
-               reading. -->
-          <mean>0.0</mean>
-          <stddev>0.01</stddev>
-        </noise>
-      </ray>
-      <plugin filename="libgazebo_ros_laser.so" name="gazebo_ros_head_hokuyo_controller">
-        <topicName>/udacity_bot/laser/scan</topicName>
-        <frameName>hokuyo</frameName>
-      </plugin>
-    </sensor>
-  </gazebo>
-  <gazebo reference="back_caster">
-    <mu1>0.0</mu1>
-    <mu2>0.0</mu2>
-  </gazebo>
-  <gazebo reference="front_caster">
-    <mu1>0.0</mu1>
-    <mu2>0.0</mu2>
-  </gazebo>
+  <!-- <xacro:include filename="$(find udacity_bot)/urdf/udacity_bot.gazebo" /> -->
   <link name="robot_footprint"/>
   <link name="chassis">
@@ -110,5 +17,5 @@
       <origin rpy=" 0 0 0" xyz="0 0 0"/>
       <geometry>
-        <box size=".4 .2 .1"/>
+        <cylinder length=".15" radius=".3"/>
       </geometry>
     </collision>
@@ -116,5 +23,5 @@
       <origin rpy=" 0 0 0" xyz="0 0 0"/>
       <geometry>
-        <box size=".4 .2 .1"/>
+        <cylinder length=".15" radius=".3"/>
       </geometry>
       <material name="black_metal">
@@ -122,10 +29,8 @@
       </material>
     </visual>
-  </link>
-  <link name="front_caster">
     <collision name="front_caster_collision">
-      <origin rpy=" 0 0 0" xyz="0.15 0 -0.05"/>
+      <origin rpy=" 0 0 0" xyz="0.15 0 -0.07"/>
       <geometry>
-        <sphere radius="0.0499"/>
+        <sphere radius="0.065"/>
       </geometry>
       <surface>
@@ -141,34 +46,7 @@
     </collision>
     <visual name="front_caster_visual">
-      <origin rpy=" 0 0 0" xyz="0.15 0 -0.05"/>
+      <origin rpy=" 0 0 0" xyz="0.15 0 -0.07"/>
       <geometry>
-        <sphere radius="0.0499"/>
-      </geometry>
-      <material name="black_metal">
-        <color rgba="0.1 0.1 0.1 1"/>
-      </material>
-    </visual>
-  </link>
-  <link name="back_caster">
-    <collision name="back_caster_collision">
-      <origin rpy=" 0 0 0" xyz="-0.15 0 -0.05"/>
-      <geometry>
-        <sphere radius="0.0498"/>
-      </geometry>
-      <surface>
-        <friction>
-          <ode>
-            <mu>0</mu>
-            <mu2>0</mu2>
-            <slip1>1.0</slip1>
-            <slip2>1.0</slip2>
-          </ode>
-        </friction>
-      </surface>
-    </collision>
-    <visual name="back_caster_visual">
-      <origin rpy=" 0 0 0" xyz="-0.15 0 -0.05"/>
-      <geometry>
-        <sphere radius="0.0498"/>
+        <sphere radius="0.065"/>
       </geometry>
       <material name="black_metal">
@@ -184,13 +62,13 @@
     </inertial>
     <collision name="left_wheel_collision">
-      <origin rpy=" 0 1.5707 1.5707" xyz="0 0 0"/>
+      <origin rpy="0 1.5707 1.5707" xyz="-0.1 0.2 -0.075"/>
       <geometry>
-        <cylinder length=".05" radius=".1"/>
+        <cylinder length=".06" radius=".05"/>
       </geometry>
     </collision>
     <visual name="left_wheel_visual">
-      <origin rpy=" 0 1.5707 1.5707" xyz="0 0 0"/>
+      <origin rpy="0 1.5707 1.5707" xyz="-0.1 0.2 -0.075"/>
       <geometry>
-        <cylinder length=".05" radius=".1"/>
+        <cylinder length=".06" radius=".05"/>
       </geometry>
     </visual>
@@ -206,13 +84,13 @@
     </inertial>
     <collision name="right_wheel_collision">
-      <origin rpy=" 0 1.5707 1.5707" xyz="0 0 0"/>
+      <origin rpy="0 1.5707 1.5707" xyz="-0.1 -0.2 -0.075"/>
       <geometry>
-        <cylinder length=".05" radius=".1"/>
+        <cylinder length=".06" radius=".05"/>
       </geometry>
     </collision>
     <visual name="right_wheel_visual">
-      <origin rpy=" 0 1.5707 1.5707" xyz="0 0 0"/>
+      <origin rpy="0 1.5707 1.5707" xyz="-0.1 -0.2 -0.075"/>
       <geometry>
-        <cylinder length=".05" radius=".1"/>
+        <cylinder length=".06" radius=".05"/>
       </geometry>
       <material name="gold">
@@ -230,5 +108,5 @@
       <origin rpy=" 0 0 0" xyz="0 0 0"/>
       <geometry>
-        <box size=".05 .05 .05"/>
+        <cylinder length=".025" radius=".025"/>
       </geometry>
     </collision>
@@ -236,5 +114,5 @@
       <origin rpy=" 0 0 0" xyz="0 0 0"/>
       <geometry>
-        <box size=".05 .05 .05"/>
+        <cylinder length=".025" radius=".025"/>
       </geometry>
     </visual>
@@ -271,5 +149,5 @@
   </joint>
   <joint name="left_wheel_hinge" type="continuous">
-    <origin rpy="0 0 0" xyz="0 0.15 0"/>
+    <origin rpy="0 0 0" xyz="0 0.15 -0.1"/>
     <parent link="chassis"/>
     <child link="left_wheel"/>
@@ -279,5 +157,5 @@
   </joint>
   <joint name="right_wheel_hinge" type="continuous">
-    <origin rpy="0 0 0" xyz="0 -0.15 0"/>
+    <origin rpy="0 0 0" xyz="0 -0.15 -0.1"/>
     <parent link="chassis"/>
     <child link="right_wheel"/>
@@ -286,19 +164,11 @@
     <joint_properties damping="1.0" friction="1.0"/>
   </joint>
-  <joint name="front_caster_hinge" type="continuous">
-    <parent link="chassis"/>
-    <child link="front_caster"/>
-  </joint>
-  <joint name="back_caster_hinge" type="continuous">
-    <parent link="chassis"/>
-    <child link="back_caster"/>
-  </joint>
   <joint name="camera_joint" type="fixed">
-    <origin rpy=" 0 0 0" xyz="0.2 0 0"/>
+    <origin rpy="0.3 0 0" xyz="0 1.5 0"/>
     <parent link="chassis"/>
     <child link="camera"/>
   </joint>
   <joint name="hokuyo_joint" type="fixed">
-    <origin rpy=" 0 0 0" xyz="0.15 0 0.2"/>
+    <origin rpy=" 0 0 0" xyz="0.15 0 0.08"/>
     <parent link="chassis"/>
     <child link="hokuyo"/>

File: urdf/udacity_bot.xacro (robot description, xacro)
@@ -2,10 +2,13 @@
 <robot name="udacity_bot" xmlns:xacro="http://www.ros.org/wiki/xacro">
 <xacro:include filename="$(find udacity_bot)/urdf/udacity_bot.gazebo" />
-  <link name="robot_footprint"></link>
+  <link name="robot_footprint">
+    <origin xyz="0 0 0" rpy=" 0 0 0"/>
+  </link>
   <link name='chassis'>
-    <pose>0 0 0.1 0 0 0</pose>
+    <origin xyz="0 0 0" rpy=" 0 0 0"/>
+    <pose>0 0 0 0 0 0</pose>
     <inertial>
       <mass value="15.0"/>
-      <origin xyz="0.0 0 0" rpy=" 0 0 0"/>
+      <origin xyz="0 0 0" rpy=" 0 0 0"/>
       <inertia
           ixx="0.2125" ixy="0" ixz="0"
@@ -17,5 +20,5 @@
       <origin xyz="0 0 0" rpy=" 0 0 0"/>
       <geometry>
-        <box size=".4 .2 .1"/>
+        <cylinder radius=".3" length=".15"/>
       </geometry>
     </collision>
@@ -23,12 +26,25 @@
       <origin xyz="0 0 0" rpy=" 0 0 0"/>
       <geometry>
-        <box size=".4 .2 .1"/>
-      </geometry>
-      <material name="black_metal">
-	<color rgba="0.1 0.1 0.1 1"/>
-      </material>
-    </visual>
+        <cylinder radius=".3" length=".15"/>
+      </geometry>
+      <material name="black_metal">
+	<color rgba="0.1 0.1 0.1 1"/>
+      </material>
+    </visual>
+  </link>
+  <link name='front_caster'>
+    <pose>0 0 0 0 0 0</pose>
+    <origin xyz="0.15 0 -0.10" rpy=" 0 0 0"/>
+    <inertial>
+    <origin xyz="0.15 0 -0.10" rpy=" 0 0 0"/>
+      <mass value="2.0"/>
+      <inertia
+          ixx="0.046" ixy="0" ixz="0"
+          iyy="0.046" iyz="0"
+          izz="0.025"
+      />
+    </inertial>
     <collision name='front_caster_collision'>
-      <origin xyz="0.15 0 -0.05" rpy=" 0 0 0"/>
+      <origin xyz="0 0 0" rpy=" 0 0 0"/>
       <geometry>
         <sphere radius="0.05"/>
@@ -46,5 +62,5 @@
     </collision>
     <visual name='front_caster_visual'>
-      <origin xyz="0.15 0 -0.05" rpy=" 0 0 0"/>
+      <origin xyz="0 0 0" rpy=" 0 0 0"/>
       <geometry>
         <sphere radius="0.05"/>
@@ -54,34 +70,11 @@
       </material>
     </visual>
-    <collision name='back_caster_collision'>
-      <origin xyz="-0.15 0 -0.05" rpy=" 0 0 0"/>
-      <geometry>
-        <sphere radius="0.05"/>
-      </geometry>
-      <surface>
-        <friction>
-          <ode>
-            <mu>0</mu>
-            <mu2>0</mu2>
-            <slip1>1.0</slip1>
-            <slip2>1.0</slip2>
-          </ode>
-        </friction>
-      </surface>
-    </collision>
-    <visual name='back_caster_visual'>
-      <origin xyz="-0.15 0 -0.05" rpy=" 0 0 0"/>
-      <geometry>
-        <sphere radius="0.05"/>
-      </geometry>
-      <material name="black_metal">
-	<color rgba="0.1 0.1 0.1 1"/>
-      </material>
-    </visual>
   </link>
   <link name='left_wheel'>
-    <inertial>
-      <mass value="5.0"/>
-      <origin xyz="0.0 0 0" rpy=" 0 0 0"/>
+    <pose>0 0 0 0 0 0</pose>
+    <origin xyz="-0.25 0.2 -0.05" rpy=" 0 0 0"/>
+    <inertial>
+    <origin xyz="-0.25 0.2 -0.05" rpy=" 0 0 0"/>
+      <mass value="2.0"/>
       <inertia
           ixx="0.046" ixy="0" ixz="0"
@@ -91,13 +84,13 @@
     </inertial>
     <collision name='left_wheel_collision'>
-      <origin xyz="0 0 0" rpy=" 0 1.5707 1.5707"/>
-      <geometry>
-        <cylinder radius=".1" length=".05"/>
+      <origin xyz="0 0 0" rpy="0 1.57 1.57"/>
+      <geometry>
+        <cylinder radius=".05" length=".06"/>
       </geometry>
     </collision>
     <visual name='left_wheel_visual'>
-      <origin xyz="0 0 0" rpy=" 0 1.5707 1.5707"/>
-      <geometry>
-        <cylinder radius=".1" length=".05"/>
+      <origin xyz="0 0 0" rpy="0 1.57 1.57"/>
+      <geometry>
+        <cylinder radius=".05" length=".06"/>
       </geometry>
     </visual>
@@ -107,7 +100,10 @@
   </link>
   <link name='right_wheel'>
-    <inertial>
-      <mass value="5.0"/>
-      <origin xyz="0.0 0 0" rpy=" 0 0 0"/>
+    <pose>0 0 0 0 0 0</pose>
+    <origin xyz="-0.25 -0.2 0.05" rpy="0 0 0"/>
+    <inertial>
+    <origin xyz="-0.25 -0.2 0.05" rpy="0 0 0"/>
+      <mass value="2.0"/>
+      <origin xyz="-0.12 -0.2 0.05" rpy="0 0 0"/>
       <inertia
           ixx="0.046" ixy="0" ixz="0"
@@ -117,13 +113,13 @@
     </inertial>
     <collision name='right_wheel_collision'>
-      <origin xyz="0 0 0" rpy=" 0 1.5707 1.5707"/>
-      <geometry>
-        <cylinder radius=".1" length=".05"/>
+      <origin xyz="0 0 0" rpy="0 1.57 1.57"/>
+      <geometry>
+        <cylinder radius=".05" length=".06"/>
       </geometry>
     </collision>
     <visual name='right_wheel_visual'>
-      <origin xyz="0 0 0" rpy=" 0 1.5707 1.5707"/>
-      <geometry>
-        <cylinder radius=".1" length=".05"/>
+      <origin xyz="0 0 0" rpy="0 1.57 1.57"/>
+      <geometry>
+        <cylinder radius=".05" length=".06"/>
       </geometry>
       <material name="gold">
@@ -133,7 +129,8 @@
   </link>
   <link name="camera">
-    <inertial>
+    <origin xyz="0.3 0 0" rpy=" 0 1.57 0"/>
+    <inertial>
+    <origin xyz="0.3 0 0" rpy=" 0 1.57 0"/>
       <mass value="0.1"/>
-      <origin xyz="0.0 0 0" rpy=" 0 0 0"/>
       <inertia
           ixx="1e-6" ixy="0" ixz="0"
@@ -145,5 +142,5 @@
       <origin xyz="0 0 0" rpy=" 0 0 0"/>
       <geometry>
-        <box size=".05 .05 .05"/>
+        <cylinder radius=".025" length=".025"/>
       </geometry>
     </collision>
@@ -151,5 +148,5 @@
       <origin xyz="0 0 0" rpy=" 0 0 0"/>
       <geometry>
-        <box size=".05 .05 .05"/>
+        <cylinder radius=".025" length=".025"/>
       </geometry>
     </visual>
@@ -159,4 +156,5 @@
   </link>
   <link name="hokuyo">
+    <origin xyz="0 0 0" rpy=" 0 0 0"/>
     <inertial>
       <mass value="0.1"/>
@@ -184,11 +182,19 @@
       </material>
   </link>
-  <joint name="robot_footprint_joint" type="fixed">
+  <joint name="chassis" type="fixed">
     <origin xyz="0 0 0" rpy="0 0 0" />
     <parent link="robot_footprint"/>
     <child link="chassis" />
   </joint>
+   <joint type="continuous" name="caster_hinge">
+       <origin xyz="0 0.15 -0.1" rpy="0 0 0"/>
+       <parent link="chassis"/>
+       <child link="front_caster"/>
+       <axis xyz="0 1 0" rpy="0 0 0"/>
+       <limit effort="10000" velocity="1000"/>
+       <joint_properties damping="1.0" friction="1.0"/>
+   </joint>
    <joint type="continuous" name="left_wheel_hinge">
-       <origin xyz="0 0.15 0" rpy="0 0 0"/>
+       <origin xyz="0 0.15 -0.1" rpy="0 0 0"/>
        <parent link="chassis"/>
        <child link="left_wheel"/>
@@ -198,5 +204,5 @@
    </joint>
    <joint type="continuous" name="right_wheel_hinge">
-       <origin xyz="0 -0.15 0" rpy="0 0 0"/>
+       <origin xyz="0 -0.15 -0.1" rpy="0 0 0"/>
        <parent link="chassis"/>
        <child link="right_wheel"/>
@@ -205,13 +211,13 @@
        <joint_properties damping="1.0" friction="1.0"/>
    </joint>
-<joint type="fixed" name="camera_joint">
-      <origin xyz="0.2 0 0" rpy=" 0 0 0"/>
+   <joint type="fixed" name="camera_joint">
+      <origin xyz="0 1.5 0" rpy="0.3 0 0"/>
       <parent link="chassis"/>
       <child link="camera"/>
-</joint>
-<joint type="fixed" name="hokuyo_joint">
+   </joint>
+   <joint type="fixed" name="hokuyo_joint">
       <origin xyz="0.15 0 0.08" rpy=" 0 0 0"/>
       <parent link="chassis"/>
       <child link="hokuyo"/>
-</joint>
+   </joint>
 </robot>
