Commit message: test

File: urdf/udacity_bot.xacro (robot description, xacro)
@@ -9,7 +9,7 @@
       <origin xyz="0.0 0 0" rpy=" 0 0 0"/>
       <inertia
-          ixx="0.1" ixy="0" ixz="0"
-          iyy="0.1" iyz="0"
-          izz="0.1"
+          ixx="0.2125" ixy="0" ixz="0"
+          iyy="0.0625" iyz="0"
+          izz="0.25"
       />
     </inertial>
@@ -29,6 +29,6 @@
       </material>
     </visual>
-    <collision name='back_caster_collision'>
-      <origin xyz="-0.15 0 -0.05" rpy=" 0 0 0"/>
+    <collision name='front_caster_collision'>
+      <origin xyz="0.15 0 -0.05" rpy=" 0 0 0"/>
       <geometry>
         <sphere radius="0.05"/>
@@ -45,12 +45,15 @@
       </surface>
     </collision>
-    <visual name='back_caster_visual'>
+    <visual name='front_caster_visual'>
+      <origin xyz="0.15 0 -0.05" rpy=" 0 0 0"/>
+      <geometry>
+        <sphere radius="0.05"/>
+      </geometry>
+      <material name="black_metal">
+	<color rgba="0.1 0.1 0.1 1"/>
+      </material>
+    </visual>
+    <collision name='back_caster_collision'>
       <origin xyz="-0.15 0 -0.05" rpy=" 0 0 0"/>
-      <geometry>
-        <sphere radius="0.05"/>
-      </geometry>
-    </visual>
-    <collision name='front_caster_collision'>
-      <origin xyz="0.15 0 -0.05" rpy=" 0 0 0"/>
       <geometry>
         <sphere radius="0.05"/>
@@ -67,9 +70,12 @@
       </surface>
     </collision>
-    <visual name='front_caster_visual'>
-      <origin xyz="0.15 0 -0.05" rpy=" 0 0 0"/>
-      <geometry>
-        <sphere radius="0.05"/>
-      </geometry>
+    <visual name='back_caster_visual'>
+      <origin xyz="-0.15 0 -0.05" rpy=" 0 0 0"/>
+      <geometry>
+        <sphere radius="0.05"/>
+      </geometry>
+      <material name="black_metal">
+	<color rgba="0.1 0.1 0.1 1"/>
+      </material>
     </visual>
   </link>
@@ -79,7 +85,7 @@
       <origin xyz="0.0 0 0" rpy=" 0 0 0"/>
       <inertia
-          ixx="0.1" ixy="0" ixz="0"
-          iyy="0.1" iyz="0"
-          izz="0.1"
+          ixx="0.046" ixy="0" ixz="0"
+          iyy="0.046" iyz="0"
+          izz="0.025"
       />
     </inertial>
@@ -96,4 +102,7 @@
       </geometry>
     </visual>
+      <material name="gold">
+        <color rgba="1 0.549 0 1"/>
+      </material>
   </link>
   <link name='right_wheel'>
@@ -102,7 +111,7 @@
       <origin xyz="0.0 0 0" rpy=" 0 0 0"/>
       <inertia
-          ixx="0.1" ixy="0" ixz="0"
-          iyy="0.1" iyz="0"
-          izz="0.1"
+          ixx="0.046" ixy="0" ixz="0"
+          iyy="0.046" iyz="0"
+          izz="0.025"
       />
     </inertial>
@@ -118,4 +127,7 @@
         <cylinder radius=".1" length=".05"/>
       </geometry>
+      <material name="gold">
+        <color rgba="1 0.549 0 1"/>
+      </material>
     </visual>
   </link>
@@ -142,4 +154,7 @@
       </geometry>
     </visual>
+      <material name="black_metal">
+	<color rgba="0.1 0.1 0.1 1"/>
+      </material>
   </link>
   <link name="hokuyo">
@@ -162,8 +177,10 @@
       <origin xyz="0 0 0" rpy=" 0 0 0"/>
       <geometry>
-        <box size=".1 .1 .1"/>
         <mesh filename="package://udacity_bot/meshes/hokuyo.dae"/>
       </geometry>
     </visual>
+      <material name="black_metal">
+	<color rgba="0.1 0.1 0.1 1"/>
+      </material>
   </link>
   <joint name="robot_footprint_joint" type="fixed">
@@ -194,5 +211,5 @@
 </joint>
 <joint type="fixed" name="hokuyo_joint">
-      <origin xyz="0.15 0 0.1" rpy=" 0 0 0"/>
+      <origin xyz="0.15 0 0.08" rpy=" 0 0 0"/>
       <parent link="chassis"/>
       <child link="hokuyo"/>

Commit message: finished own gazebo model

File: urdf/udacity_bot.xacro (robot description, xacro)
@@ -6,6 +6,5 @@
   </link>
   <link name='chassis'>
-    <origin xyz="0 0 0" rpy=" 0 0 0"/>
-    <pose>0 0 0 0 0 0</pose>
+    <pose>0 0 0.3 0 0 0</pose>
     <inertial>
       <mass value="15.0"/>
@@ -32,10 +31,18 @@
       </material>
     </visual>
+    <visual name='chassis_dome_visual'>
+      <origin xyz="0 0 0.1" rpy=" 0 0 0"/>
+      <geometry>
+        <cylinder radius=".05" length=".05"/>
+      </geometry>
+      <material name="black_metal">
+	<color rgba="0.1 0.1 0.1 1"/>
+      </material>
+    </visual>
   </link>
   <link name='front_caster'>
     <pose>0 0 0 0 0 0</pose>
-    <origin xyz="0.15 0 -0.10" rpy=" 0 0 0"/>
-    <inertial>
-    <origin xyz="0.15 0 -0.10" rpy=" 0 0 0"/>
+    <inertial>
+      <origin xyz="0 0 0" rpy=" 0 0 0"/>
       <mass value="2.0"/>
       <inertia
@@ -73,7 +80,6 @@
   <link name='left_wheel'>
     <pose>0 0 0 0 0 0</pose>
-    <origin xyz="-0.25 0.2 -0.05" rpy=" 0 0 0"/>
-    <inertial>
-    <origin xyz="-0.25 0.2 -0.05" rpy=" 0 0 0"/>
+    <inertial>
+      <origin xyz="0 0 0" rpy="0 1.57 1.57"/>
       <mass value="2.0"/>
       <inertia
@@ -101,9 +107,7 @@
   <link name='right_wheel'>
     <pose>0 0 0 0 0 0</pose>
-    <origin xyz="-0.25 -0.2 0.05" rpy="0 0 0"/>
-    <inertial>
-    <origin xyz="-0.25 -0.2 0.05" rpy="0 0 0"/>
+    <inertial>
+      <origin xyz="0 0 0" rpy="0 1.57 1.57"/>
       <mass value="2.0"/>
-      <origin xyz="-0.12 -0.2 0.05" rpy="0 0 0"/>
       <inertia
           ixx="0.046" ixy="0" ixz="0"
@@ -129,7 +133,6 @@
   </link>
   <link name="camera">
-    <origin xyz="0.3 0 0" rpy=" 0 1.57 0"/>
-    <inertial>
-    <origin xyz="0.3 0 0" rpy=" 0 1.57 0"/>
+    <inertial>
+    <origin xyz="0 0 0" rpy=" 0 0 0"/>
       <mass value="0.1"/>
       <inertia
@@ -156,5 +159,4 @@
   </link>
   <link name="hokuyo">
-    <origin xyz="0 0 0" rpy=" 0 0 0"/>
     <inertial>
       <mass value="0.1"/>
@@ -183,10 +185,10 @@
   </link>
   <joint name="chassis" type="fixed">
-    <origin xyz="0 0 0" rpy="0 0 0" />
+    <origin xyz="0 0 0.3" rpy="0 0 0" />
     <parent link="robot_footprint"/>
     <child link="chassis" />
   </joint>
    <joint type="continuous" name="caster_hinge">
-       <origin xyz="0 0.15 -0.1" rpy="0 0 0"/>
+       <origin xyz="0.2 0 -0.05" rpy="0 0 0"/>
        <parent link="chassis"/>
        <child link="front_caster"/>
@@ -196,5 +198,5 @@
    </joint>
    <joint type="continuous" name="left_wheel_hinge">
-       <origin xyz="0 0.15 -0.1" rpy="0 0 0"/>
+       <origin xyz="-0.15 0.15 -0.05" rpy="0 0 0"/>
        <parent link="chassis"/>
        <child link="left_wheel"/>
@@ -204,5 +206,5 @@
    </joint>
    <joint type="continuous" name="right_wheel_hinge">
-       <origin xyz="0 -0.15 -0.1" rpy="0 0 0"/>
+       <origin xyz="-0.15 -0.15 -0.05" rpy="0 0 0"/>
        <parent link="chassis"/>
        <child link="right_wheel"/>
@@ -212,10 +214,10 @@
    </joint>
    <joint type="fixed" name="camera_joint">
-      <origin xyz="0 1.5 0" rpy="0.3 0 0"/>
+      <origin xyz="0.3 0 0" rpy=" 0 1.57 0"/>
       <parent link="chassis"/>
       <child link="camera"/>
    </joint>
    <joint type="fixed" name="hokuyo_joint">
-      <origin xyz="0.15 0 0.08" rpy=" 0 0 0"/>
+      <origin xyz="0 0 0.15" rpy=" 0 0 0"/>
       <parent link="chassis"/>
       <child link="hokuyo"/>

Commit message: further parameter tuning

File: urdf/udacity_bot.xacro (robot description, xacro)
@@ -11,7 +11,7 @@
       <origin xyz="0 0 0" rpy=" 0 0 0"/>
       <inertia
-          ixx="0.2125" ixy="0" ixz="0"
-          iyy="0.0625" iyz="0"
-          izz="0.25"
+          ixx="0.365625" ixy="0" ixz="0"
+          iyy="0.365625" iyz="0"
+          izz="0.675"
       />
     </inertial>
@@ -47,7 +47,7 @@
       <mass value="2.0"/>
       <inertia
-          ixx="0.046" ixy="0" ixz="0"
-          iyy="0.046" iyz="0"
-          izz="0.025"
+          ixx="0.002" ixy="0" ixz="0"
+          iyy="0.002" iyz="0"
+          izz="0.002"
       />
     </inertial>
@@ -84,7 +84,7 @@
       <mass value="2.0"/>
       <inertia
-          ixx="0.046" ixy="0" ixz="0"
-          iyy="0.046" iyz="0"
-          izz="0.025"
+          ixx="0.00185" ixy="0" ixz="0"
+          iyy="0.00185" iyz="0"
+          izz="0.0025"
       />
     </inertial>
@@ -111,7 +111,7 @@
       <mass value="2.0"/>
       <inertia
-          ixx="0.046" ixy="0" ixz="0"
-          iyy="0.046" iyz="0"
-          izz="0.025"
+          ixx="0.00185" ixy="0" ixz="0"
+          iyy="0.00185" iyz="0"
+          izz="0.0025"
       />
     </inertial>
@@ -214,5 +214,5 @@
    </joint>
    <joint type="fixed" name="camera_joint">
-      <origin xyz="0.3 0 0" rpy=" 0 1.57 0"/>
+      <origin xyz="0.3 0 0" rpy="1.57 1.57 0"/>
       <parent link="chassis"/>
       <child link="camera"/>

Commit message: wheel redesign was a breakthrough - robot finally behaves

File: urdf/udacity_bot.xacro (robot description, xacro)
@@ -6,8 +6,8 @@
   </link>
   <link name='chassis'>
-    <pose>0 0 0.3 0 0 0</pose>
+    <pose>0 0 0 0 0 0</pose>
     <inertial>
       <mass value="15.0"/>
-      <origin xyz="0 0 0" rpy=" 0 0 0"/>
+      <origin xyz="0 0 -0.05" rpy="0 0 0"/>
       <inertia
           ixx="0.365625" ixy="0" ixz="0"
@@ -17,5 +17,5 @@
     </inertial>
     <collision name='chassis_collision'>
-      <origin xyz="0 0 0" rpy=" 0 0 0"/>
+      <origin xyz="0 0 .015" rpy=" 0 0 0"/>
       <geometry>
         <cylinder radius=".3" length=".15"/>
@@ -23,5 +23,5 @@
     </collision>
     <visual name='chassis_visual'>
-      <origin xyz="0 0 0" rpy=" 0 0 0"/>
+      <origin xyz="0 0 .015" rpy=" 0 0 0"/>
       <geometry>
         <cylinder radius=".3" length=".15"/>
@@ -32,5 +32,5 @@
     </visual>
     <visual name='chassis_dome_visual'>
-      <origin xyz="0 0 0.1" rpy=" 0 0 0"/>
+      <origin xyz="-0.2 0 0.11" rpy=" 0 0 0"/>
       <geometry>
         <cylinder radius=".05" length=".05"/>
@@ -78,4 +78,41 @@
     </visual>
   </link>
+  <link name='back_caster'>
+    <pose>0 0 0 0 0 0</pose>
+    <inertial>
+      <origin xyz="0 0 0" rpy=" 0 0 0"/>
+      <mass value="2.0"/>
+      <inertia
+          ixx="0.002" ixy="0" ixz="0"
+          iyy="0.002" iyz="0"
+          izz="0.002"
+      />
+    </inertial>
+    <collision name='back_caster_collision'>
+      <origin xyz="0 0 0" rpy=" 0 0 0"/>
+      <geometry>
+        <sphere radius="0.05"/>
+      </geometry>
+      <surface>
+        <friction>
+          <ode>
+            <mu>0</mu>
+            <mu2>0</mu2>
+            <slip1>1.0</slip1>
+            <slip2>1.0</slip2>
+          </ode>
+        </friction>
+      </surface>
+    </collision>
+    <visual name='back_caster_visual'>
+      <origin xyz="0 0 0" rpy=" 0 0 0"/>
+      <geometry>
+        <sphere radius="0.05"/>
+      </geometry>
+      <material name="black_metal">
+	<color rgba="0.1 0.1 0.1 1"/>
+      </material>
+    </visual>
+  </link>
   <link name='left_wheel'>
     <pose>0 0 0 0 0 0</pose>
@@ -185,9 +222,9 @@
   </link>
   <joint name="chassis" type="fixed">
-    <origin xyz="0 0 0.3" rpy="0 0 0" />
+    <origin xyz="0 0 0" rpy="0 0 0" />
     <parent link="robot_footprint"/>
     <child link="chassis" />
   </joint>
-   <joint type="continuous" name="caster_hinge">
+   <joint type="continuous" name="front_caster_hinge">
        <origin xyz="0.2 0 -0.05" rpy="0 0 0"/>
        <parent link="chassis"/>
@@ -197,6 +234,14 @@
        <joint_properties damping="1.0" friction="1.0"/>
    </joint>
+   <joint type="continuous" name="back_caster_hinge">
+       <origin xyz="-0.2 0 -0.05" rpy="0 0 0"/>
+       <parent link="chassis"/>
+       <child link="back_caster"/>
+       <axis xyz="0 1 0" rpy="0 0 0"/>
+       <limit effort="10000" velocity="1000"/>
+       <joint_properties damping="1.0" friction="1.0"/>
+   </joint>
    <joint type="continuous" name="left_wheel_hinge">
-       <origin xyz="-0.15 0.15 -0.05" rpy="0 0 0"/>
+       <origin xyz="0 0.2 -0.05" rpy="0 0 0"/>
        <parent link="chassis"/>
        <child link="left_wheel"/>
@@ -206,5 +251,5 @@
    </joint>
    <joint type="continuous" name="right_wheel_hinge">
-       <origin xyz="-0.15 -0.15 -0.05" rpy="0 0 0"/>
+       <origin xyz="0 -0.2 -0.05" rpy="0 0 0"/>
        <parent link="chassis"/>
        <child link="right_wheel"/>
@@ -214,10 +259,10 @@
    </joint>
    <joint type="fixed" name="camera_joint">
-      <origin xyz="0.3 0 0" rpy="1.57 1.57 0"/>
+      <origin xyz="0.3 0 0" rpy="0.075 1.57 0.075"/>
       <parent link="chassis"/>
       <child link="camera"/>
    </joint>
    <joint type="fixed" name="hokuyo_joint">
-      <origin xyz="0 0 0.15" rpy=" 0 0 0"/>
+      <origin xyz="-0.2 0 0.16" rpy=" 0 0 0"/>
       <parent link="chassis"/>
       <child link="hokuyo"/>

Commit message: got rtabmap running

File: urdf/udacity_bot.xacro (robot description, xacro)
@@ -169,5 +169,5 @@
     </visual>
   </link>
-  <link name="camera">
+  <link name="camera_link">
     <inertial>
     <origin xyz="0 0 0" rpy=" 0 0 0"/>
@@ -195,4 +195,5 @@
       </material>
   </link>
+  <link name="camera_rgbd_frame" />
   <link name="hokuyo">
     <inertial>
@@ -261,5 +262,10 @@
       <origin xyz="0.3 0 0" rpy="0.075 1.57 0.075"/>
       <parent link="chassis"/>
-      <child link="camera"/>
+      <child link="camera_link"/>
+   </joint>
+   <joint type="fixed" name="rgbd_camera_joint">
+      <orign xyz="0 0 0" rpy="${-pi/2} 0 ${-pi/2}"/>
+      <parent link="camera_link"/>
+      <child link="camera_rgbd_frame"/>
    </joint>
    <joint type="fixed" name="hokuyo_joint">

Commit message: map floating in the air, but overall good progess

File: urdf/udacity_bot.xacro (robot description, xacro)
@@ -171,5 +171,5 @@
   <link name="camera_link">
     <inertial>
-    <origin xyz="0 0 0" rpy=" 0 0 0"/>
+    <origin xyz="0 0 0" rpy="0 0 0"/>
       <mass value="0.1"/>
       <inertia
@@ -182,5 +182,5 @@
       <origin xyz="0 0 0" rpy=" 0 0 0"/>
       <geometry>
-        <cylinder radius=".025" length=".025"/>
+        <box size="0.05 0.05 0.05"/>
       </geometry>
     </collision>
@@ -188,12 +188,13 @@
       <origin xyz="0 0 0" rpy=" 0 0 0"/>
       <geometry>
-        <cylinder radius=".025" length=".025"/>
-      </geometry>
-    </visual>
-      <material name="black_metal">
-	<color rgba="0.1 0.1 0.1 1"/>
-      </material>
-  </link>
-  <link name="camera_rgbd_frame" />
+        <box size="0.05 0.05 0.05"/>
+        <!--<cylinder radius=".025" length=".025"/>-->
+      </geometry>
+    </visual>
+      <material name="black_metal">
+	<color rgba="0.1 0.1 0.1 1"/>
+      </material>
+  </link>
+  <link name="camera_link_optical" />
   <link name="hokuyo">
     <inertial>
@@ -260,12 +261,12 @@
    </joint>
    <joint type="fixed" name="camera_joint">
-      <origin xyz="0.3 0 0" rpy="0.075 1.57 0.075"/>
+      <origin xyz="0.3 0 0" rpy="0 0 0"/>
       <parent link="chassis"/>
       <child link="camera_link"/>
    </joint>
-   <joint type="fixed" name="rgbd_camera_joint">
-      <orign xyz="0 0 0" rpy="${-pi/2} 0 ${-pi/2}"/>
+   <joint type="fixed" name="camera_rgbd_joint">
+      <orign xyz="0.3 0 0" rpy="${-pi/2} 0 ${-pi/2}"/>
       <parent link="camera_link"/>
-      <child link="camera_rgbd_frame"/>
+      <child link="camera_link_optical"/>
    </joint>
    <joint type="fixed" name="hokuyo_joint">

Commit message: still struggeling with the pointcloud

File: urdf/udacity_bot.xacro (robot description, xacro)
@@ -10,9 +10,5 @@
       <mass value="15.0"/>
       <origin xyz="0 0 -0.05" rpy="0 0 0"/>
-      <inertia
-          ixx="0.365625" ixy="0" ixz="0"
-          iyy="0.365625" iyz="0"
-          izz="0.675"
-      />
+      <inertia ixx="0.365625" ixy="0" ixz="0" iyy="0.365625" iyz="0" izz="0.675" />
     </inertial>
     <collision name='chassis_collision'>
@@ -41,4 +37,9 @@
     </visual>
   </link>
+  <joint name="chassis" type="fixed">
+    <origin xyz="0 0 0" rpy="0 0 0" />
+    <parent link="robot_footprint"/>
+    <child link="chassis" />
+  </joint>
   <link name='front_caster'>
     <pose>0 0 0 0 0 0</pose>
@@ -46,9 +47,5 @@
       <origin xyz="0 0 0" rpy=" 0 0 0"/>
       <mass value="2.0"/>
-      <inertia
-          ixx="0.002" ixy="0" ixz="0"
-          iyy="0.002" iyz="0"
-          izz="0.002"
-      />
+      <inertia ixx="0.002" ixy="0" ixz="0" iyy="0.002" iyz="0" izz="0.002" />
     </inertial>
     <collision name='front_caster_collision'>
@@ -78,4 +75,12 @@
     </visual>
   </link>
+   <joint type="continuous" name="front_caster_hinge">
+       <origin xyz="0.2 0 -0.05" rpy="0 0 0"/>
+       <parent link="chassis"/>
+       <child link="front_caster"/>
+       <axis xyz="0 1 0" rpy="0 0 0"/>
+       <limit effort="10000" velocity="1000"/>
+       <joint_properties damping="1.0" friction="1.0"/>
+   </joint>
   <link name='back_caster'>
     <pose>0 0 0 0 0 0</pose>
@@ -115,4 +120,12 @@
     </visual>
   </link>
+   <joint type="continuous" name="back_caster_hinge">
+       <origin xyz="-0.2 0 -0.05" rpy="0 0 0"/>
+       <parent link="chassis"/>
+       <child link="back_caster"/>
+       <axis xyz="0 1 0" rpy="0 0 0"/>
+       <limit effort="10000" velocity="1000"/>
+       <joint_properties damping="1.0" friction="1.0"/>
+   </joint>
   <link name='left_wheel'>
     <pose>0 0 0 0 0 0</pose>
@@ -120,9 +133,5 @@
       <origin xyz="0 0 0" rpy="0 1.57 1.57"/>
       <mass value="2.0"/>
-      <inertia
-          ixx="0.00185" ixy="0" ixz="0"
-          iyy="0.00185" iyz="0"
-          izz="0.0025"
-      />
+      <inertia ixx="0.00185" ixy="0" ixz="0" iyy="0.00185" iyz="0" izz="0.0025" />
     </inertial>
     <collision name='left_wheel_collision'>
@@ -142,4 +151,12 @@
       </material>
   </link>
+   <joint type="continuous" name="left_wheel_hinge">
+       <origin xyz="0 0.2 -0.05" rpy="0 0 0"/>
+       <parent link="chassis"/>
+       <child link="left_wheel"/>
+       <axis xyz="0 1 0" rpy="0 0 0"/>
+       <limit effort="10000" velocity="1000"/>
+       <joint_properties damping="1.0" friction="1.0"/>
+   </joint>
   <link name='right_wheel'>
     <pose>0 0 0 0 0 0</pose>
@@ -147,9 +164,5 @@
       <origin xyz="0 0 0" rpy="0 1.57 1.57"/>
       <mass value="2.0"/>
-      <inertia
-          ixx="0.00185" ixy="0" ixz="0"
-          iyy="0.00185" iyz="0"
-          izz="0.0025"
-      />
+      <inertia ixx="0.00185" ixy="0" ixz="0" iyy="0.00185" iyz="0" izz="0.0025" />
     </inertial>
     <collision name='right_wheel_collision'>
@@ -169,13 +182,18 @@
     </visual>
   </link>
+   <joint type="continuous" name="right_wheel_hinge">
+       <origin xyz="0 -0.2 -0.05" rpy="0 0 0"/>
+       <parent link="chassis"/>
+       <child link="right_wheel"/>
+       <axis xyz="0 1 0" rpy="0 0 0"/>
+       <limit effort="10000" velocity="1000"/>
+       <joint_properties damping="1.0" friction="1.0"/>
+   </joint>
   <link name="camera_link">
-    <inertial>
     <origin xyz="0 0 0" rpy="0 0 0"/>
+    <inertial>
       <mass value="0.1"/>
-      <inertia
-          ixx="1e-6" ixy="0" ixz="0"
-          iyy="1e-6" iyz="0"
-          izz="1e-6"
-      />
+      <origin xyz="0 0 0" rpy="0 0 0"/>
+      <inertia ixx="1e-6" ixy="0" ixz="0" iyy="1e-6" iyz="0" izz="1e-6" />
     </inertial>
     <collision name='camera_collision'>
@@ -189,12 +207,23 @@
       <geometry>
         <box size="0.05 0.05 0.05"/>
-        <!--<cylinder radius=".025" length=".025"/>-->
-      </geometry>
-    </visual>
-      <material name="black_metal">
-	<color rgba="0.1 0.1 0.1 1"/>
-      </material>
-  </link>
+      </geometry>
+    </visual>
+  </link>
+   <joint type="fixed" name="camera_joint">
+      <origin xyz="0.3 0 0" rpy="0 0 0"/>
+      <child link="camera_link"/>
+      <parent link="chassis"/>
+      <axis xyz="0 1 0" rpy="0 0 0"/>
+    <!--
+    <limit effort="10000" velocity="1000"/>
+    <dynamics damping="1.0" friction="1.0"/>
+    -->
+   </joint>
   <link name="camera_link_optical" />
+   <joint type="fixed" name="camera_optical_joint">
+      <orign xyz="0.3 0 0" rpy="-1.5707 0 -1.5707"/>
+      <parent link="camera_link"/>
+      <child link="camera_link_optical"/>
+   </joint>
   <link name="hokuyo">
     <inertial>
@@ -202,8 +231,5 @@
       <origin xyz="0.0 0 0" rpy=" 0 0 0"/>
       <inertia
-          ixx="1e-6" ixy="0" ixz="0"
-          iyy="1e-6" iyz="0"
-          izz="1e-6"
-      />
+          ixx="1e-6" ixy="0" ixz="0" iyy="1e-6" iyz="0" izz="1e-6" />
     </inertial>
     <collision name='hokuyo_collision'>
@@ -223,51 +249,4 @@
       </material>
   </link>
-  <joint name="chassis" type="fixed">
-    <origin xyz="0 0 0" rpy="0 0 0" />
-    <parent link="robot_footprint"/>
-    <child link="chassis" />
-  </joint>
-   <joint type="continuous" name="front_caster_hinge">
-       <origin xyz="0.2 0 -0.05" rpy="0 0 0"/>
-       <parent link="chassis"/>
-       <child link="front_caster"/>
-       <axis xyz="0 1 0" rpy="0 0 0"/>
-       <limit effort="10000" velocity="1000"/>
-       <joint_properties damping="1.0" friction="1.0"/>
-   </joint>
-   <joint type="continuous" name="back_caster_hinge">
-       <origin xyz="-0.2 0 -0.05" rpy="0 0 0"/>
-       <parent link="chassis"/>
-       <child link="back_caster"/>
-       <axis xyz="0 1 0" rpy="0 0 0"/>
-       <limit effort="10000" velocity="1000"/>
-       <joint_properties damping="1.0" friction="1.0"/>
-   </joint>
-   <joint type="continuous" name="left_wheel_hinge">
-       <origin xyz="0 0.2 -0.05" rpy="0 0 0"/>
-       <parent link="chassis"/>
-       <child link="left_wheel"/>
-       <axis xyz="0 1 0" rpy="0 0 0"/>
-       <limit effort="10000" velocity="1000"/>
-       <joint_properties damping="1.0" friction="1.0"/>
-   </joint>
-   <joint type="continuous" name="right_wheel_hinge">
-       <origin xyz="0 -0.2 -0.05" rpy="0 0 0"/>
-       <parent link="chassis"/>
-       <child link="right_wheel"/>
-       <axis xyz="0 1 0" rpy="0 0 0"/>
-       <limit effort="10000" velocity="1000"/>
-       <joint_properties damping="1.0" friction="1.0"/>
-   </joint>
-   <joint type="fixed" name="camera_joint">
-      <origin xyz="0.3 0 0" rpy="0 0 0"/>
-      <parent link="chassis"/>
-      <child link="camera_link"/>
-   </joint>
-   <joint type="fixed" name="camera_rgbd_joint">
-      <orign xyz="0.3 0 0" rpy="${-pi/2} 0 ${-pi/2}"/>
-      <parent link="camera_link"/>
-      <child link="camera_link_optical"/>
-   </joint>
    <joint type="fixed" name="hokuyo_joint">
       <origin xyz="-0.2 0 0.16" rpy=" 0 0 0"/>
