Commit message: mapped provided environment

File: urdf/udacity_bot.xacro (robot description, xacro)
@@ -37,9 +37,45 @@
     </visual>
   </link>
-  <joint name="chassis" type="fixed">
+  <joint name="chassis_joint" type="fixed">
     <origin xyz="0 0 0" rpy="0 0 0" />
     <parent link="robot_footprint"/>
     <child link="chassis" />
   </joint>
+  <link name="camera_link">
+    <origin xyz="0 0 0" rpy="0 0 0"/>
+    <inertial>
+      <mass value="0.1"/>
+      <origin xyz="0 0 0" rpy="0 0 0"/>
+      <inertia ixx="1e-6" ixy="0" ixz="0" iyy="1e-6" iyz="0" izz="1e-6" />
+    </inertial>
+    <collision name='camera_collision'>
+      <origin xyz="0 0 0" rpy=" 0 0 0"/>
+      <geometry>
+        <box size="0.05 0.05 0.05"/>
+      </geometry>
+    </collision>
+    <visual name='camera_visual'>
+      <origin xyz="0 0 0" rpy=" 0 0 0"/>
+      <geometry>
+        <box size="0.05 0.05 0.05"/>
+      </geometry>
+    </visual>
+  </link>
+   <joint name="camera_joint" type="fixed">
+      <origin xyz="0.3 0 0" rpy="0 0 0"/>
+      <child link="camera_link"/>
+      <parent link="chassis"/>
+      <axis xyz="0 1 0" rpy="0 0 0"/>
+    <!--
+    <limit effort="10000" velocity="1000"/>
+    <dynamics damping="1.0" friction="1.0"/>
+    -->
+   </joint>
+  <link name="camera_link_optical"></link>
+   <joint name="camera_optical_joint" type="fixed" >
+      <origin xyz="0.3 0 0" rpy="-1.5707 0 -1.5707"/>
+      <parent link="camera_link"/>
+      <child link="camera_link_optical"/>
+   </joint>
   <link name='front_caster'>
     <pose>0 0 0 0 0 0</pose>
@@ -190,40 +226,4 @@
        <joint_properties damping="1.0" friction="1.0"/>
    </joint>
-  <link name="camera_link">
-    <origin xyz="0 0 0" rpy="0 0 0"/>
-    <inertial>
-      <mass value="0.1"/>
-      <origin xyz="0 0 0" rpy="0 0 0"/>
-      <inertia ixx="1e-6" ixy="0" ixz="0" iyy="1e-6" iyz="0" izz="1e-6" />
-    </inertial>
-    <collision name='camera_collision'>
-      <origin xyz="0 0 0" rpy=" 0 0 0"/>
-      <geometry>
-        <box size="0.05 0.05 0.05"/>
-      </geometry>
-    </collision>
-    <visual name='camera_visual'>
-      <origin xyz="0 0 0" rpy=" 0 0 0"/>
-      <geometry>
-        <box size="0.05 0.05 0.05"/>
-      </geometry>
-    </visual>
-  </link>
-   <joint type="fixed" name="camera_joint">
-      <origin xyz="0.3 0 0" rpy="0 0 0"/>
-      <child link="camera_link"/>
-      <parent link="chassis"/>
-      <axis xyz="0 1 0" rpy="0 0 0"/>
-    <!--
-    <limit effort="10000" velocity="1000"/>
-    <dynamics damping="1.0" friction="1.0"/>
-    -->
-   </joint>
-  <link name="camera_link_optical" />
-   <joint type="fixed" name="camera_optical_joint">
-      <orign xyz="0.3 0 0" rpy="-1.5707 0 -1.5707"/>
-      <parent link="camera_link"/>
-      <child link="camera_link_optical"/>
-   </joint>
   <link name="hokuyo">
     <inertial>
